Commit message: feat: deploy V15.17 inertial parameters

File: V15_14_MoveIt2_ROS2_Control_MuJoCo_轨迹闭环/ros2_ws/src/go_m8010_arm_v15_14_description/urdf/go_m8010_arm_v15_14.urdf.xacro (robot description, xacro)
@@ -48,4 +48,9 @@
   </link>
   <link name="link2">
+    <inertial>
+      <origin xyz="-0.09682602754229415 -0.01627177564337673 0.00026852096508443425" rpy="0 0 0" />
+      <mass value="0.7615" />
+      <inertia ixx="0.0011506145878779188" ixy="-0.0009540393634177025" ixz="9.404715830688318e-06" iyy="0.007217558727290144" iyz="6.257421623983668e-06" izz="0.007407791096012893" />
+    </inertial>
     <visual>
       <origin xyz="0 0 0" rpy="0 0 0" />
@@ -57,4 +62,9 @@
   </link>
   <link name="link3">
+    <inertial>
+      <origin xyz="-0.10115006408445788 0.034091146941368534 0.02591627514565488" rpy="0 0 0" />
+      <mass value="1.09" />
+      <inertia ixx="0.0014953205051949686" ixy="-3.464298746690975e-06" ixz="0.0027501824929620057" iyy="0.012662694095746066" iyz="2.570114870295044e-06" izz="0.01145498720138968" />
+    </inertial>
     <visual>
       <origin xyz="0 0 0" rpy="0 0 0" />
@@ -66,4 +76,9 @@
   </link>
   <link name="link4">
+    <inertial>
+      <origin xyz="-0.003256288062399695 0.026691901325969727 0.07712273077803503" rpy="0 0 0" />
+      <mass value="0.675" />
+      <inertia ixx="0.0017846928666986044" ixy="5.576191808676761e-06" ixz="3.260540608689319e-05" iyy="0.0014691530030288575" iyz="-0.0002629908074224898" izz="0.0004889558170829342" />
+    </inertial>
     <visual>
       <origin xyz="0 0 0" rpy="0 0 0" />
@@ -75,4 +90,9 @@
   </link>
   <link name="link5">
+    <inertial>
+      <origin xyz="-0.007314793455186482 -0.0001338266798615075 0.06388991222545329" rpy="0 0 0" />
+      <mass value="0.504" />
+      <inertia ixx="0.0006923549323153038" ixy="-3.23074993999531e-07" ixz="0.00011373297010931771" iyy="0.0007038092568726869" iyz="7.950330868652517e-07" izz="0.0003002790321734546" />
+    </inertial>
     <visual>
       <origin xyz="0 0 0" rpy="0 0 0" />
@@ -84,4 +104,9 @@
   </link>
   <link name="link6">
+    <inertial>
+      <origin xyz="-1.1047636330058231e-15 1.360430323081585e-16 -0.0005011957785718855" rpy="0 0 0" />
+      <mass value="0.125" />
+      <inertia ixx="1.1518299692789527e-05" ixy="8.646775045799554e-20" ixz="1.7766902612207907e-18" iyy="1.1518299692790563e-05" iyz="-5.319523438636526e-21" izz="2.3015838872973936e-05" />
+    </inertial>
     <visual>
       <origin xyz="0 0 0" rpy="0 0 0" />
@@ -93,4 +118,9 @@
   </link>
   <link name="gripper">
+    <inertial>
+      <origin xyz="-0.0034049824167213345 -0.0007997027279568269 0.03493651236222258" rpy="0 0 0" />
+      <mass value="0.296" />
+      <inertia ixx="0.00045010858437538907" ixy="5.241520235144432e-06" ixz="-3.6621915682408926e-05" iyy="0.00037548194776002844" iyz="-6.980811698347642e-07" izz="0.0004173108380272847" />
+    </inertial>
     <visual>
       <origin xyz="0 0 0" rpy="0 0 0" />
